File: PCB-V01/mapleSDuino-V0.1_010-eagle7.sch (EAGLE design)
At the start: 11 parts, among them IC2 LAN-USR-ES1

Commit message: V010
Parts:
- removed U$2: CC1101_MODULE1DIL_BIG, CC1101:CC1101_MODULE1DIL_BIG
- added TRX3, TX3: (no value), SparkFun-Connectors:CONN_04PTH
- DBG: device con-lstb:MA04-1 -> SparkFun-Connectors:CONN_04LOCK
- EXT: device con-lstb:MA04-1 -> SparkFun-Connectors:CONN_04PTH
Connections:
- net WIZ_CS renamed SS2
- removed net N$33: IC2.!INT!
- removed net RST: IC2.MOSI, U$1.28/SPI2_MOSI
- removed net RX_DBG: DBG.3, U$1.25/PWM/RX1
- removed net TX_DBG: DBG.2, U$1.26/PWM/TX1
- new net MOSI2: CC1.MOSI, CC2.MOSI, TRX3.3, U$1.28/SPI2_MOSI
- new net SS1: U$1.7/AIN/SPI1_SS
- net CC_CS0: no longer U$1.7/AIN/SPI1_SS
- net CC_CS2: now also TX3.4; no longer U$2.CSN
- net CC_IN_2: now also TX3.2; no longer U$2.GDO2
- net CC_OUT_2: now also TX3.3; no longer U$2.GDO0
- net GND: now also TRX3.2; no longer U$2.GND@1, U$2.GND@2, U$2.GND@3
- net MISO1: now also IC2.MISO; no longer CC1.MISO, CC2.MISO, U$2.MISO
- net MISO2: now also CC1.MISO, CC2.MISO, TX3.1; no longer IC2.MISO
- net MOSI1: now also IC2.MOSI; no longer CC1.MOSI, CC2.MOSI, U$2.MOSI
- net RX1: now also DBG.3, U$1.25/PWM/RX1
- net SCK1: now also IC2.SCLK; no longer CC1.SCLK, CC2.SCLK, U$2.SCLK
- net SCK2: now also CC1.SCLK, CC2.SCLK, TRX3.4; no longer IC2.SCLK
- net TX1: now also DBG.2, U$1.26/PWM/TX1
- net VCC: now also TRX3.1; no longer U$2.VCC
Other:
- moved on the sheet: IC2
