File: PCB-V01/mapleSDuino-V0.1_012-eagle7.brd (EAGLE design)
At the start: 79 x 27 mm, 23 parts, among them IC2 LAN-USR-ES1

Commit message: Fix CS
Parts:
- removed CC2: CC1101_MODULE1SMD, wireless:CC1101_MODULE1_SMD
- added CC0: CC1101, wireless:CC1101_MODULE1_SMD
- CC1: value CC1101 -> CC1101_MODULE1SMD
- moved CC1 22.9 mm to (57.1, 24.8), flipped to the bottom, turned to 180 degrees
- moved TP8 0.74 mm to (77.6, 8.76)
- moved TP10 0.63 mm to (77.6, 14.7)
- moved TP7 0.63 mm to (77.6, 25.4)
- moved TP9 0.38 mm to (54.9, 8.76)
Connections:
- removed net SS2: CC1.CSN, CC2.CSN, TX3.4, U$1.20
- new net CC_CS0: CC0.CSN
- net ANT1: now also CC1.ANT; no longer CC2.ANT
- net ANT2: now also CC0.ANT; no longer CC1.ANT
- net CC_CS1: now also CC1.CSN, U$1.20
- net CC_CS2: now also TX3.4
- net CC_IN_0: now also CC0.GDO2; no longer CC1.GDO2
- net CC_IN_1: now also CC1.GDO2; no longer CC2.GDO2
- net CC_OUT_0: now also CC0.GDO0; no longer CC1.GDO0
- net CC_OUT_1: now also CC1.GDO0; no longer CC2.GDO0
- net GND: now also CC0.GND@0, CC0.GND@1, CC0.GND@2; no longer CC2.GND@0, CC2.GND@1, CC2.GND@2
- net MISO2: now also CC0.MISO; no longer CC2.MISO
- net MOSI2: now also CC0.MOSI; no longer CC2.MOSI
- net SCK2: now also CC0.SCLK; no longer CC2.SCLK
- net VCC: now also CC0.VCC; no longer CC2.VCC
Routing:
- net GND: track 272.2 -> 0.00 mm, vias 1 -> 0
- net VCC: track 140.9 -> 0.00 mm, vias 1 -> 0
- net MISO2: track 73.9 -> 0.00 mm, vias 1 -> 0
- net MOSI1: track 60.5 -> 0.00 mm
- net SS2: track 58.7 -> 0.00 mm, vias 1 -> 0
- net CC_OUT_1: track 45.0 -> 0.00 mm, vias 1 -> 0
- net SCK2: track 44.6 -> 0.00 mm, vias 1 -> 0
- net CC_IN_1: track 40.9 -> 0.00 mm, vias 1 -> 0
- net CC_IN_0: track 38.6 -> 0.00 mm
- net CC_OUT_0: track 37.2 -> 0.00 mm
- net MOSI2: track 36.3 -> 0.00 mm, vias 1 -> 0
- net CC_IN_2: track 32.0 -> 0.00 mm
- net WIZ_RST: track 30.1 -> 0.00 mm
- net MISO1: track 29.6 -> 0.00 mm
- net +5V: track 29.4 -> 0.00 mm, vias 2 -> 0
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Other:
- board text added: "MapleSDuino"
