File: PCB-V01/mapleSDuino-V0.1_012-eagle7.sch (EAGLE design)
At the start: 23 parts, among them IC2 LAN-USR-ES1

Commit message: Fix CS
Parts:
- removed CC2: CC1101_MODULE1SMD, wireless:CC1101_MODULE1SMD
- added CC0: CC1101, wireless:CC1101_MODULE1SMD
- CC1: value CC1101 -> CC1101_MODULE1SMD
Connections:
- removed net SS2: CC1.CSN, CC2.CSN, TX3.4, U$1.31/SPI2_SS
- new net CC_CS0: CC0.CSN
- net ANT1: now also CC1.ANT; no longer CC2.ANT
- net ANT2: now also CC0.ANT; no longer CC1.ANT
- net CC_CS1: now also CC1.CSN, U$1.31/SPI2_SS
- net CC_CS2: now also TX3.4
- net CC_IN_0: now also CC0.GDO2; no longer CC1.GDO2
- net CC_IN_1: now also CC1.GDO2; no longer CC2.GDO2
- net CC_OUT_0: now also CC0.GDO0; no longer CC1.GDO0
- net CC_OUT_1: now also CC1.GDO0; no longer CC2.GDO0
- net GND: now also CC0.GND@1, CC0.GND@2, CC0.GND@3; no longer CC2.GND@1, CC2.GND@2, CC2.GND@3
- net MISO2: now also CC0.MISO; no longer CC2.MISO
- net MOSI2: now also CC0.MOSI; no longer CC2.MOSI
- net SCK2: now also CC0.SCLK; no longer CC2.SCLK
- net VCC: now also CC0.VCC; no longer CC2.VCC
Other:
- note added: "LAN, ..."
- note added: "Shielding (not needed, but pussible)"
- note removed: "LAN"
- note removed: "siehe Homematic"
- note removed: "siehe MySensors"
- moved on the sheet: CC1, EXT, IC2, TP1, TP10, TP11, TP2, TP3, TP4, TP5, TP6, TP7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
