File: PCB-V01/mapleSDuino-V0.1_013-eagle7.brd (EAGLE design)
At the start: 79 x 27 mm, 23 parts, among them IC2 LAN-USR-ES1

Commit message: pin 31
Connections:
- net CC_CS0: now also U$1.20
- net CC_CS1: no longer U$1.20
Changed lines of the file:
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@@
 <contactref element="U$1" pad="35"/>
 <contactref element="CC1" pad="CSN"/>
-<contactref element="U$1" pad="20"/>
-<wire x1="52.705" y1="20.955" x2="57.15" y2="24.765" width="0" layer="19" extent="16-16"/>
-<wire x1="17.145" y1="5.715" x2="52.705" y2="20.955" width="0" layer="19" extent="1-1"/>
+<wire x1="17.145" y1="5.715" x2="57.15" y2="24.765" width="0" layer="19" extent="16-16"/>
 </signal>
 <signal name="CC_IN_1">
@@
 <signal name="CC_CS0">
 <contactref element="CC0" pad="CSN"/>
+<contactref element="U$1" pad="20"/>
+<wire x1="57.15" y1="1.905" x2="52.705" y2="20.955" width="0" layer="19" extent="1-1"/>
 </signal>
 </signals>
