File: PCB-V01/mapleSDuino-V0.1_013-eagle7.sch (EAGLE design)
At the start: 23 parts, among them IC2 LAN-USR-ES1

Commit message: pin 31
Connections:
- net CC_CS0: now also U$1.31/SPI2_SS
- net CC_CS1: no longer U$1.31/SPI2_SS
Changed lines of the file:
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@@
 <label x="175.26" y="220.98" size="1.778" layer="95"/>
-</segment>
-<segment>
-<pinref part="U$1" gate="G$1" pin="31/SPI2_SS"/>
-<wire x1="133.35" y1="113.03" x2="116.84" y2="113.03" width="0.1524" layer="91"/>
-<label x="124.46" y="113.03" size="1.778" layer="95"/>
 </segment>
 </net>
@@
 <label x="100.33" y="220.98" size="1.778" layer="95"/>
 </segment>
+<segment>
+<pinref part="U$1" gate="G$1" pin="31/SPI2_SS"/>
+<wire x1="133.35" y1="113.03" x2="116.84" y2="113.03" width="0.1524" layer="91"/>
+<label x="124.46" y="113.03" size="1.778" layer="95"/>
+</segment>
 </net>
