File: PCB-V01/mapleSDuino-V0.1_014-eagle7.brd (EAGLE design)
At the start: 79 x 27 mm, 23 parts, among them IC2 LAN-USR-ES1

Commit message: Labels Part1
Parts:
- moved X1 0.63 mm to (81.9, 6.99)
Other:
- outline, holes or cut-outs redrawn
- board text added: "10uF"
- board text added: "5V"
- board text added: "CC2"
- board text added: "CS2"
- board text added: "DBG"
- board text added: "EXT"
- board text added: "IN2"
- board text added: "MISO2"
- board text added: "MOSI"
- board text added: "OUT2"
- board text added: "SCK"
- board text added: "V 0.1 (C) www.neuby.de"
- board text removed: "MAPLE CUL"
- board text removed: "Small V2.0 www.neuby.de"
