File: PCB-V01/mapleSDuino-V0.1_019-eagle7.brd (EAGLE design)
At the start: 79 x 27 mm, 23 parts, among them IC2 LAN-USR-ES1

Commit message: 019
Parts:
- added TP12, TP13, TP14, TP15: TPTP06SQ, testpad:TP06SQ
- moved TP6 21.8 mm to (54.9, 3.30)
- moved TP9 20.9 mm to (66.0, 26.4)
- moved C5 9.94 mm to (27.9, 15.2), turned to 90 degrees
- moved C6 4.13 mm to (14.0, 17.8), turned to 180 degrees
- moved IC2 2.54 mm to (14.0, 13.3)
- moved EXT 2.54 mm to (43.2, 2.54)
- moved X2 0.40 mm to (81.8, 20.6), flipped to the bottom, turned to 0 degrees
- moved X1 0.18 mm to (81.8, 6.86)
- renumbered TRX3 to CC3A, TX3 to CC3B
Connections:
- net GND: now also TP12.TP, TP13.TP, TP14.TP, TP15.TP
Routing:
- net GND: track 0.00 -> 272.1 mm, vias 0 -> 3
- net VCC: track 0.00 -> 127.6 mm, vias 0 -> 3
- net MISO2: track 0.00 -> 65.4 mm, vias 0 -> 1
- net CC_CS1: track 0.00 -> 49.2 mm, vias 0 -> 1
- net CC_OUT_1: track 0.00 -> 45.4 mm, vias 0 -> 1
- net CC_IN_0: track 0.00 -> 44.0 mm
- net SCK2: track 0.00 -> 41.5 mm, vias 0 -> 1
- net CC_IN_1: track 0.00 -> 41.4 mm, vias 0 -> 1
- net MOSI2: track 0.00 -> 39.3 mm, vias 0 -> 1
- net CC_OUT_0: track 0.00 -> 37.2 mm, vias 0 -> 1
- net CC_CS2: track 0.00 -> 33.5 mm
- net MOSI1: track 0.00 -> 32.3 mm, vias 0 -> 1
- net CC_IN_2: track 0.00 -> 32.2 mm, vias 0 -> 1
- net WIZ_RST: track 0.00 -> 27.5 mm
- net SCK1: track 0.00 -> 27.2 mm, vias 0 -> 1
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Other:
- board text added: "433 MHz"
- board text added: "868 MHz"
- board text added: "V0.1 www.neuby.de"
- board text removed: "10uF"
- board text removed: "CC0"
- board text removed: "CC2"
- board text removed: "DBG"
- board text removed: "EXT"
