File: PCB-V01/mapleSDuino-V0.1_019-eagle7.sch (EAGLE design)
At the start: 23 parts, among them IC2 LAN-USR-ES1

Commit message: 019
Parts:
- added TP12, TP13, TP14, TP15: TPTP06SQ, testpad:TPTP06SQ
- renumbered TRX3 to CC3A, TX3 to CC3B
Connections:
- net GND: now also TP12.TP, TP13.TP, TP14.TP, TP15.TP
Other:
- note added: "Shielding (not needed, but possible)"
- note removed: "Shielding (not needed, but pussible)"
- moved on the sheet: EXT, IC2, TP1, TP10, TP11, TP2, TP3, TP5, TP6, TP7, TP9
