File: PCB-V01/mapleSDuino-V0.1_020-eagle7.brd (EAGLE design)
At the start: 79 x 27 mm, 27 parts, among them IC2 LAN-USR-ES1

Commit message: V01-final
Routing:
- net GND: vias 3 -> 30
Changed lines of the file:
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@@
 <setting verticaltext="up"/>
 </settings>
-<grid distance="10" unitdist="mil" unit="mil" style="dots" multiple="1" display="yes" altdistance="0.025" altunitdist="inch" altunit="inch"/>
+<grid distance="5" unitdist="mil" unit="mil" style="dots" multiple="1" display="yes" altdistance="0.025" altunitdist="inch" altunit="inch"/>
 <layers>
 <layer number="1" name="Top" color="2" fill="1" visible="yes" active="yes"/>
@@
 <wire x1="77.3683" y1="23.114" x2="77.3683" y2="24.5158" width="0.4064" layer="16"/>
 <wire x1="77.3683" y1="24.5158" x2="77.597" y2="24.7445" width="0.4064" layer="16"/>
+<via x="16.002" y="10.922" extent="1-16" drill="0.6" shape="square"/>
+<via x="4.826" y="2.286" extent="1-16" drill="0.6" shape="square"/>
+<via x="4.572" y="25.4" extent="1-16" drill="0.6" shape="square"/>
+<via x="24.384" y="24.384" extent="1-16" drill="0.6" shape="square"/>
+<via x="80.01" y="25.654" extent="1-16" drill="0.6" shape="square"/>
+<via x="75.692" y="25.654" extent="1-16" drill="0.6" shape="square"/>
+<via x="72.898" y="25.654" extent="1-16" drill="0.6" shape="square"/>
+<via x="79.883" y="2.159" extent="1-16" drill="0.6" shape="square"/>
+<via x="74.803" y="2.159" extent="1-16" drill="0.6" shape="square"/>
+<via x="69.723" y="2.159" extent="1-16" drill="0.6" shape="square"/>
+<via x="60.198" y="1.524" extent="1-16" drill="0.6" shape="square"/>
+<via x="39.243" y="2.794" extent="1-16" drill="0.6" shape="square"/>
+<via x="46.863" y="12.319" extent="1-16" drill="0.6" shape="square"/>
+<via x="40.513" y="14.224" extent="1-16" drill="0.6" shape="square"/>
+<via x="60.833" y="22.479" extent="1-16" drill="0.6" shape="square"/>
+<via x="60.833" y="18.669" extent="1-16" drill="0.6" shape="square"/>
+<via x="60.833" y="14.859" extent="1-16" drill="0.6" shape="square"/>
+<via x="60.833" y="10.414" extent="1-16" drill="0.6" shape="square"/>
+<via x="60.833" y="6.604" extent="1-16" drill="0.6" shape="square"/>
+<via x="72.263" y="6.604" extent="1-16" drill="0.6" shape="square"/>
+<via x="72.263" y="10.414" extent="1-16" drill="0.6" shape="square"/>
+<via x="72.263" y="14.859" extent="1-16" drill="0.6" shape="square"/>
+<via x="72.263" y="18.669" extent="1-16" drill="0.6" shape="square"/>
+<via x="72.263" y="21.209" extent="1-16" drill="0.6" shape="square"/>
+<via x="48.768" y="8.509" extent="1-16" drill="0.6" shape="square"/>
+<via x="24.003" y="2.159" extent="1-16" drill="0.6" shape="square"/>
+<via x="24.257" y="12.827" extent="1-16" drill="0.6" shape="square"/>
 </signal>
 <signal name="+5V" class="1">
@@
 <contactref element="CC0" pad="ANT"/>
 <contactref element="X1" pad="P"/>
-<wire x1="79.756" y1="6.858" x2="78.749" y2="7.865" width="0.3048" layer="1"/>
-<wire x1="78.749" y1="7.865" x2="76.15" y2="7.865" width="0.3048" layer="1"/>
+<wire x1="76.15" y1="7.865" x2="79.121" y2="6.731" width="0.4064" layer="1"/>
+<wire x1="79.121" y1="6.731" x2="79.756" y2="6.858" width="0.4064" layer="1"/>
 </signal>
 <signal name="ANT1" class="1">
 <contactref element="CC1" pad="ANT"/>
 <contactref element="X2" pad="P"/>
-<wire x1="79.756" y1="20.574" x2="77.3683" y2="20.574" width="0.4064" layer="16"/>
-<wire x1="77.3683" y1="20.574" x2="77.3683" y2="20.0233" width="0.4064" layer="16"/>
-<wire x1="77.3683" y1="20.0233" x2="76.15" y2="18.805" width="0.4064" layer="16"/>
+<wire x1="76.15" y1="18.805" x2="77.089" y2="19.05" width="0.4064" layer="16"/>
+<wire x1="77.089" y1="19.05" x2="78.105" y2="20.193" width="0.4064" layer="16"/>
+<wire x1="78.105" y1="20.193" x2="79.756" y2="20.574" width="0.4064" layer="16"/>
 </signal>
 <signal name="SS1">
