File: PCB-V09/mapleSDuino-V0.9_014-eagle7-test.brd (EAGLE design)
At the start: 79 x 27 mm, 24 parts, among them IC2 LAN-USR-ES1

Commit message: V0.9
Parts:
- CC0: device Martin-Communication-V4:CC1101_MODULE1_SMD -> CC1101:CC1101_MODULE1_SMD
- CC1: value CC1101_MODULE1SMALL -> CC1101_MODULE1SMD; device Martin-Communication-V4:CC1101_MODULE1_SMD -> CC1101:CC1101_MODULE1_SMD
- moved DBG 21.6 mm to (43.2, 2.54)
- moved EXT 21.6 mm to (43.2, 24.1)
Routing:
- net TX1: track 13.6 -> 38.2 mm, vias 0 -> 1
- net RX1: track 18.9 -> 43.1 mm, vias 0 -> 1
- net GND: track 316.0 -> 295.3 mm, vias 52 -> 27
- net +5V: track 29.4 -> 14.9 mm
- net MISO2: track 69.9 -> 57.8 mm, vias 2 -> 1
- net CC_OUT_2: track 25.6 -> 33.1 mm, vias 0 -> 1
- net CC_CS0: track 34.4 -> 27.5 mm
- net SCK2: track 48.1 -> 41.3 mm, vias 1 -> 2
- net RX2: track 23.5 -> 30.2 mm
- net MOSI2: track 39.4 -> 33.5 mm
- net CC_CS1: track 59.1 -> 64.7 mm
- net CC_OUT_1: track 45.3 -> 49.9 mm
- net ANT2: track 7.95 -> 4.02 mm
- net ANT1: track 7.91 -> 4.34 mm
- net TX2: track 26.0 -> 29.2 mm, vias 1 -> 0
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Other:
- board text added: "(C) www.neuby.de"
- board text added: "MapleSDuino V0.9"
- board text added: "V 0.9"
- board text removed: "V 0.9 (C) www.neuby.de"
- board text removed: "V0.9 www.neuby.de"
