File: PCB-V09/mapleSDuino-V0.9_014-eagle7-test.sch (EAGLE design)
At the start: 24 parts, among them IC2 LAN-USR-ES1

Commit message: V0.9
Parts:
- CC0: device Martin-Communication-V4:CC1101_MODULE1SMALL -> CC1101:CC1101_MODULE1SMD
- CC1: value CC1101_MODULE1SMALL -> CC1101_MODULE1SMD; device Martin-Communication-V4:CC1101_MODULE1SMALL -> CC1101:CC1101_MODULE1SMD
Changed lines of the file:
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@@
 <parts>
 <part name="U$1" library="maplemini-small" deviceset="MAPLEMINI" device=""/>
-<part name="CC1" library="Martin-Communication-V4" deviceset="CC1101_MODULE1" device="SMALL"/>
+<part name="CC1" library="CC1101" deviceset="CC1101_MODULE1" device="SMD"/>
 <part name="GND3" library="supply1" deviceset="GND" device=""/>
 <part name="GND4" library="supply1" deviceset="GND" device=""/>
@@
 <part name="SUPPLY1" library="supply2" deviceset="VCC" device=""/>
 <part name="GND1" library="supply1" deviceset="GND" device=""/>
-<part name="CC0" library="Martin-Communication-V4" deviceset="CC1101_MODULE1" device="SMALL" value="CC1101"/>
+<part name="CC0" library="CC1101" deviceset="CC1101_MODULE1" device="SMD" value="CC1101"/>
 <part name="GND8" library="supply1" deviceset="GND" device=""/>
 <part name="GND9" library="supply1" deviceset="GND" device=""/>
